File: CHECON.PCB Design Files/CHECON.PCB.brd (EAGLE design)
At the start: 117.9 x 57.1 mm, 75 parts, among them T1 BC849, U2 MAX232SOIC16, U3 RS485SOIC, X1 53047-02

Commit message: Working on layout
Layout
Parts:
- removed POSCON, SCANNER: (no value), GW-devices:RJ45_SMD
- removed U$11, U$12, U$17, U$21, U$22, U$23, U$56, U$58, U$62: 1uF, GW-devices:C0805
- removed U$14: USB_B, KW2:USB-B-PTH-VERTICAL
- removed U$15, U$16, U$4, U$5, U$8: MIC94061C6, GW-devices:SC70-6L
- removed U$18, U$19, U$20: BCR401U, KW2:SOT23-6
- removed U$24, U$31, U$32, U$63: 10uF, GW-devices:C0805
- removed U$25, U$36, U$37, U$6: 10k, GW-devices:RF-C0805
- removed U$26: 40, GW-devices:RF-C0805
- removed U$27, U$28: 15, GW-devices:RF-C0805
- removed U$3: KL20, KW2:QFN-32
- removed U$33: 1.5k, GW-devices:RF-C0805
- removed U$34, U$60, U$61: 4.7k, GW-devices:RF-C0805
- removed U$38, U$39, U$40, U$41, U$42, U$43: (no value), adafruit:FIDUCIAL_1MM
- removed U$44: LED_PTH_2812, KW2:LED_PTH_2812
- removed U$45: PCA9632DP1, KW2:TSSOP-8
- removed U$48: 120, GW-devices:RF-C0805
- removed U$50: CJS, KW2:CJS
- removed U$53: AP5724, KW2:SOT23-6
- removed U$54: 4.99, GW-devices:RF-C0805
- removed U$55: NR4012T220M, KW2:NR4012T220M
- removed U$57: BM78, KW2:BM78
- removed U$59, U$7: 0.1uF, GW-devices:C0805
- removed U$64: CSTCE8M00G55-R0, KW2:CSTCE_G_A
- added C1, C12, C15, C2, C3, C4, C5, C6, C8: 1uF, GW-devices:C0805
- added C10, C13, C14, C9: 10uF, GW-devices:C0805
- added C11, C16: 0.1uF, GW-devices:C0805
- added D2: LED_PTH_2812, KW2:LED_PTH_2812
- added F1, F2, F3, F4, F5, F6: FIDUCIAL, adafruit:FIDUCIAL_1MM
- added J2: USB_B, KW2:USB-B-PTH-VERTICAL
- added L2: (no value), SparkFun:0603
- added P1, P2: RJ45-8PEGMOUNT, GW-devices:MOLEX-0955016889
- added R1, R14, R15, R16, R17, R3: 10k, GW-devices:RF-C0805
- added R10: 1.5k, GW-devices:RF-C0805
- added R11, R8, R9: 4.7k, GW-devices:RF-C0805
- added R2: 120, GW-devices:RF-C0805
- added R4: 4.99, GW-devices:RF-C0805
- added R5: 40, GW-devices:RF-C0805
- added R6, R7: 15, GW-devices:RF-C0805
- added SW1, SW2: CJS, KW2:CJS
- added U1: BM78, KW2:BM78
- added U11: PCA9632DP1, KW2:TSSOP-8
- added U12: KL20, KW2:QFN-32-NOPAD
- added U4: RS485SOIC, SparkFun:SO08
- added U5, U7, U8, U9: MIC94061C6, GW-devices:SC70-6L
- added U6: AP5724, KW2:SOT23-6
- added X2, X3, X4: BCR401U, KW2:SOT23-6
- added X5: CSTCE8M00G55-R0, KW2:CSTCE_G_A
- L1: value (none) -> NR4012T220M; device SparkFun:0603 -> KW2:NR4012T220M
- U3: value RS485SOIC -> MIC94061C6; device SparkFun:SO08 -> GW-devices:SC70-6L
- moved L1 48.2 mm to (18.3, -5.30)
- moved IC1 41.2 mm to (-36.8, -1.00)
- moved U3 14.6 mm to (8.38, -28.3), flipped to the bottom, turned to 270 degrees
- moved D1 6.71 mm to (21.6, -8.40), turned to 180 degrees
- moved U2 2.39 mm to (3.40, -19.7), turned to 180 degrees
- moved T1 0.82 mm to (-35.2, -18.3)
- moved X1 0.36 mm to (-11.4, -39.7)
- moved JP2 0.22 mm to (-37.6, -31.9)
- moved JP1 0.14 mm to (-11.9, -32.1)
- renumbered U$1 to J1, U$10 to U10, U$13 to D4, U$2 to J3, U$29 to C7, U$30 to S1, U$35 to R12, U$46 to C17, U$47 to R19, U$49 to R18, U$51 to SW3, U$52 to R13, U$9 to D3
Connections:
- removed net N$8: U$15.3
- new net N$24: R16.2, U12.3
- new net N$59: R2.2, SW1.P$3
- new net N$60: R17.2, U12.4
- net +3V3: now also C14.2, C15.2, C16.2, C8.2, C9.2, L1.P$2, R1.2, R11.1, R3.2, R8.1, U11.8, U12.1, U12.7, U6.6; no longer U$3.1, U$3.7, U$32.2, U$36.2, U$37.2, U$45.8, U$53.6, U$55.P$2, U$58.2, U$59.2, U$60.1, U$61.1, U$62.2, U$63.2
- net +5V: now also C10.2, D2.P$2, U7.4, U8.4, U9.4; no longer U$15.4, U$16.4, U$31.2, U$44.P$2, U$8.4
- net C1: now also C1.1; no longer U$11.1
- net C2: now also C2.1; no longer U$12.1
- net GND: now also C10.1, C11.2, C12.2, C13.2, C14.1, C15.1, C16.1, C3.2, C4.2, C5.2, C6.1, C8.1, C9.1, D2.P$3, J2.GND, L2.2, P1.P$2, P2.P$2, P2.P$7, R14.2, R15.2, R4.2, U1.P$1, U1.P$2, U1.P$3, U1.P$31, U1.P$32, U1.P$33, U11.5, U12.2, U12.8, U3.2, U4.5, U5.2, U5.5, U6.2, U7.2, U7.5, U8.2, U8.5, U9.2, U9.5, X2.1, X3.1, X4.1, X5.P$2; no longer L1.2, POSCON.P$2, POSCON.P$7, SCANNER.P$2, U$14.GND, U$15.2, U$15.5, U$16.2, U$16.5, U$17.2, U$18.1, U$19.1, U$20.1, U$21.2, U$22.2, U$23.2, U$24.2, U$25.2, U$3.2, U$3.8, U$31.1, U$32.1, U$4.2, U$4.5, U$44.P$3, U$45.5, U$5.2, U$5.5, U$53.2, U$54.2, U$56.1, U$57.P$1, U$57.P$2, U$57.P$3, U$57.P$31, U$57.P$32, U$57.P$33, U$58.1, U$59.1, U$6.2, U$62.1, U$63.1, U$64.P$2, U$7.2, U$8.2, U$8.5
- net N$1: now also SW2.P$3, U12.27, U12.28; no longer U$3.27, U$3.28, U$50.P$3
- net N$11: now also R10.2, R9.2; no longer U$33.2, U$34.2
- net N$12: now also P1.P$4; no longer SCANNER.P$4
- net N$13: now also R6.1, U9.1, X4.4; no longer U$16.1, U$20.4, U$28.1
- net N$14: now also R7.1, U8.1, X3.4; no longer U$15.1, U$19.4, U$27.1
- net N$15: now also R5.1, U7.1, X2.4; no longer U$18.4, U$26.1, U$8.1
- net N$17: now also U4.1; no longer U3.1
- net N$18: now also C1.2; no longer U$11.2
- net N$19: now also P2.P$4, R2.1, U4.7; no longer POSCON.P$4, U$48.1, U3.7
- net N$2: now also U11.2, U6.4; no longer U$45.2, U$53.4
- net N$20: now also P2.P$5, SW1.P$1, U4.6; no longer POSCON.P$5, U$48.2, U3.6
- net N$21: now also C2.2; no longer U$12.2
- net N$22: now also C5.1; no longer U$23.1
- net N$23: now also C4.1; no longer U$22.1
- net N$25: now also C3.1, P1.P$1, U3.1; no longer SCANNER.P$1, U$21.1, U$4.1
- net N$27: now also U4.4; no longer U3.4
- net N$28: now also U4.2, U4.3; no longer U3.2, U3.3
- net N$3: now also R4.1, U6.3; no longer U$53.3, U$54.1
- net N$32: now also R15.1; no longer U$6.1
- net N$33: now also R14.1; no longer U$25.1
- net N$34: now also P1.P$5; no longer SCANNER.P$5
- net N$35: now also J2.D-, R17.1; no longer U$14.D-, U$3.4
- net N$36: now also J2.D+, R16.1; no longer U$14.D+, U$3.3
- net N$37: now also R6.2, X4.6; no longer U$20.6, U$28.2
- net N$39: now also R3.1, U5.3; no longer U$36.1, U$5.3
- net N$4: now also U12.17, X5.P$1; no longer U$3.17, U$64.P$1
- net N$40: now also R1.1, U3.3; no longer U$37.1, U$4.3
- net N$42: now also R7.2, X3.6; no longer U$19.6, U$27.2
- net N$43: now also R5.2, X2.6; no longer U$18.6, U$26.2
- net N$44: now also U11.1, U7.3, U8.3, U9.3; no longer U$16.3, U$45.1, U$8.3
- net N$45: now also R11.2, U11.7; no longer U$45.7, U$61.2
- net N$47: now also R8.2, U11.6; no longer U$45.6, U$60.2
- net N$48: now also D2.P$1, R10.1; no longer U$33.1, U$44.P$1
- net N$49: now also R9.1; no longer U$34.1
- net N$5: now also J2.P$1, J2.P$2, L2.1; no longer L1.1, U$14.P$1, U$14.P$2
- net N$50: now also L1.P$1, U6.1; no longer U$53.1, U$55.P$1
- net N$51: now also X4.2, X4.3, X4.5; no longer U$20.2, U$20.3, U$20.5
- net N$52: now also U12.15; no longer U$3.15
- net N$53: now also X3.2, X3.3, X3.5; no longer U$19.2, U$19.3, U$19.5
- net N$54: now also C6.2, U6.5; no longer U$53.5, U$56.2
- net N$55: now also U12.12; no longer U$3.12
- net N$56: now also U12.14; no longer U$3.14
- net N$57: now also U12.13; no longer U$3.13
- net N$58: now also U12.19; no longer U$3.19
- net N$6: now also U12.18, X5.P$3; no longer U$3.18, U$64.P$3
- net N$7: now also P1.P$6; no longer SCANNER.P$6
- net N$9: now also X2.2, X2.3, X2.5; no longer U$18.2, U$18.3, U$18.5
- net R1IN: now also P1.P$3; no longer SCANNER.P$3
- net RST: now also U12.21; no longer U$3.21
- net SWD_DIO: now also SW2.P$1; no longer U$50.P$1
- net SWD_TGT_CLK: now also U12.26; no longer U$3.26
- net V+: now also C11.1, C12.1, C13.1, P2.P$1, P2.P$8, U3.4, U4.8, U5.1, U5.4; no longer POSCON.P$1, POSCON.P$8, U$17.1, U$24.1, U$4.4, U$5.1, U$5.4, U$7.1, U3.8
Routing:
- net GND: track 0.00 -> 70.4 mm, vias 0 -> 3
- net N$51: track 0.00 -> 60.1 mm
- net N$9: track 0.00 -> 47.0 mm
- net N$53: track 0.00 -> 28.1 mm, vias 0 -> 2
- net N$45: track 0.00 -> 26.2 mm, vias 0 -> 1
- net N$44: track 0.00 -> 24.2 mm
- net +3V3: track 0.00 -> 21.4 mm
- net N$47: track 0.00 -> 19.2 mm, vias 0 -> 1
- net +5V: track 0.00 -> 19.1 mm, vias 0 -> 3
- net V+: track 0.00 -> 17.0 mm
- net N$50: track 0.00 -> 14.0 mm
- net N$2: track 0.00 -> 13.2 mm, vias 0 -> 2
- net N$13: track 0.00 -> 10.3 mm
- net N$15: track 0.00 -> 10.1 mm
- net N$14: track 0.00 -> 10.1 mm
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Other:
- board size 117.9 x 57.1 mm -> 123.7 x 51.6 mm
