File: CHECON.PCB Design Files/CHECON.PCB.sch (EAGLE design)
At the start: 73 parts, among them U2 MAX232SOIC16, U3 RS485SOIC

Commit message: New CHE
Starting on new CHE
Parts:
- removed C11, C14: 0.1uF, GW-devices:RF-C0805
- removed LQH3NPN100NM0L: 1212_IND, KW2:1212_IND
- removed R10: (no value), GW-devices:RF-R2512
- removed R12, R13: 10, GW-devices:RF-R0805
- removed U$59: BL_CON, KW2:BL_CON
- removed U$62: INA219B, KW2:INA219B
- added D1: (no value), adafruit:DIODESOD-523
- added JP1, JP2: (no value), KW2:PINHD-2X5SMALL
- added L1: (no value), SparkFun:INDUCTOR0603
- added T1: BC849, transistor:BC849
- added X1: 53047-02, con-molex:53047-02
- U$1: value RGLBED -> 2.7_BL_CONN; device KW2:RGLBED -> KW2:2.7_BL_CONN; MFGN (none) -> Omron Electronics; MFGP (none) -> XD2B-0406-26A
- U$13: value SWITCH-TACTILE-FSM -> TVS0603; device GW-devices:SWITCH-TACTILE-FSM -> SparkFun:TVS0603; MFGN E-Switch -> Eaton Bussman; MFGP TL3301DF160QG -> 0603ESDA2-TR2
- U$14: value SWITCH-TACTILE-FSM -> USB_B; device GW-devices:SWITCH-TACTILE-FSM -> KW2:USB_B; MFGN E-Switch -> Harwin; MFGP TL3301DF160QG -> M701-330442
- U$15, U$16: value SWITCH-TACTILE-FSM -> MIC94061C6; device GW-devices:SWITCH-TACTILE-FSM -> GW-devices:MIC94061C6; MFGN E-Switch -> (none); MFGP TL3301DF160QG -> (none)
- U$18, U$19, U$20: value 24 -> BCR401U; device GW-devices:RF-R0805 -> KW2:BCR401U; MFGN Vishay Dale -> Infineon; MFGP CRCW080524R0FKEA -> BCR401U
- U$26: value 10k -> 40; MFGN Vishay Dale -> Yageo; MFGP CRCW080510K0FKEA -> RC0805FR-0740R2L
- U$27, U$28: value 10k -> 15; MFGN Vishay Dale -> Yageo; MFGP CRCW080510K0FKEA -> RC0805FR-0715RL
- U$29: value 10k -> 220pF; device GW-devices:RF-R0805 -> GW-devices:RF-C0805; MFGN Vishay Dale -> TDK; MFGP CRCW080510K0FKEA -> C2012X5R1H104K085AA
- U$3: value 2X10JTAG -> KL20; device KW2:2X10JTAG -> KW2:KL20; MFGN (none) -> Freescale; MFGP (none) -> MK20DX128VFM5
- U$33: value 0.1uF -> 1.5k; device GW-devices:RF-C0805 -> GW-devices:RF-R0805; MFGN TDK -> Vishay Dale; MFGP C2012X5R1H104K085AA -> CRCW080510K0FKEA
- U$34: value 1uF -> 4.7k; device GW-devices:RF-C0805 -> GW-devices:RF-R0805; MFGN TDK -> Vishay Dale; MFGP C2012X5R1E105K125AA -> CRCW080510K0FKEA
- U$35: value 10uF -> 1.1k; device GW-devices:RF-C0805 -> GW-devices:RF-R0805; MFGN Murata -> Vishay Dale; MFGP GRM219R61E106KA12D -> CRCW080510K0FKEA
- U$36, U$37: value SC4541 -> 10k; device KW2:SC4541 -> GW-devices:RF-R0805; MFGN (none) -> Panasonic; MFGP (none) -> ERJ-6ENF4701V
- U$44: value SC4541 -> LED_PTH_2812; device KW2:SC4541 -> KW2:LED_PTH_2812; MFGN (none) -> Sparkfun; MFGP (none) -> COM-12999
- U$46: value 10k -> 0.1uF; device GW-devices:RF-R0805 -> GW-devices:RF-C0805; MFGN Vishay Dale -> TDK; MFGP CRCW080510K0FKEA -> C2012X5R1H104K085AA
- U$47, U$49: value 1212_IND -> 10k; device KW2:1212_IND -> GW-devices:RF-R0805; MFGN Murata -> Vishay Dale; MFGP LQH3NPN100NM0L -> CRCW080510K0FKEA
- U$50, U$51: value 1uF -> CJS; device GW-devices:RF-C0805 -> KW2:CJS; MFGN TDK -> (none); MFGP C2012X5R1E105K125AA -> (none)
- U$52: value 1uF -> 10k; device GW-devices:RF-C0805 -> GW-devices:RF-R0805; MFGN TDK -> Vishay Dale; MFGP C2012X5R1E105K125AA -> CRCW080510K0FKEA
- U$53: value 1uF -> AP5724; device GW-devices:RF-C0805 -> KW2:AP5724; MFGN TDK -> Diodes, Inc; MFGP C2012X5R1E105K125AA -> AP5724
- U$54: value 1uF -> 4.99; device GW-devices:RF-C0805 -> GW-devices:RF-R0805; MFGN TDK -> Stackpole Electronics Inc.; MFGP C2012X5R1E105K125AA -> RMCF0805FT4R99
- U$55: value 1uF -> NR4012T220M; device GW-devices:RF-C0805 -> KW2:NR4012T220M; MFGN TDK -> Taiyo Yuden; MFGP C2012X5R1E105K125AA -> NR4012T220M
- U$56: value 6.8 -> 1uF; device GW-devices:RF-R0805 -> GW-devices:RF-C0805; MFGN Yageo -> TDK; MFGP RC0805FR-076R8L -> C2012X5R1E105K125AA
- U$57: value 3.3 -> BM78; device GW-devices:RF-R0805 -> KW2:BM78; MFGN Samsung -> (none); MFGP RC2012F3R3CS -> (none)
- U$58: value 3.3 -> 1uF; device GW-devices:RF-R0805 -> GW-devices:RF-C0805; MFGN Samsung -> TDK; MFGP RC2012F3R3CS -> C2012X5R1E105K125AA
- U$8: value WS2801 -> MIC94061C6; device GW-devices:WS2801 -> GW-devices:MIC94061C6; MFGP WS2801 -> (none)
- U$9: value BARREL_CUI_PJ-002A -> TVS0603; device KW2:BARREL_CUI_PJ-002A -> SparkFun:TVS0603; MFGN (none) -> Eaton Bussman; MFGP (none) -> 0603ESDA2-TR2
- U2: MFGP MAX232DR -> (none)
- U3: MFGP SN65HVD1781DR -> (none)
Connections:
- removed net N$24: POSCON.1, POSCON.8, U$5.VOUT
- new net +5V: IC1.IN, U$15.VIN, U$16.VIN, U$31.2, U$44.VDD, U$8.VIN
- new net N$58: JP2.10, U$3.RST, U$49.2
- net +3V3: now also JP1.1, JP2.1, U$36.2, U$37.2, U$46.2, U$52.1, U$53.VIN, U$55.2, U$58.2; no longer C14.1, LQH3NPN100NM0L.1, U$21.1, U$26.2, U$27.2, U$28.2, U$29.2, U$3.P$1, U$36.IN, U$37.IN, U$44.IN, U$62.VS, U2.VCC
- net GND: now also JP1.3, JP1.5, JP2.3, JP2.5, L1.2, U$1.P$4, U$14.GND, U$15.GND1, U$15.GND2, U$16.GND1, U$16.GND2, U$18.GND, U$19.GND, U$20.GND, U$29.1, U$53.GND, U$56.1, U$57.GND, U$57.GND1, U$57.GND2, U$57.GND4, U$57.GND5, U$57.GND6, U$58.1, U$8.GND1, U$8.GND2, U$9.1; no longer C14.2, U$13.2, U$14.1, U$14.2, U$15.1, U$15.2, U$16.1, U$16.2, U$18.2, U$19.2, U$20.2, U$3.P$15, U$3.P$17, U$3.P$19, U$3.P$3, U$3.P$5, U$3.P$9, U$33.1, U$34.1, U$36.GND, U$37.GND, U$50.1, U$51.1, U$52.1, U$53.2, U$55.2, U$59.GND, U$62.A0, U$62.A1, U$62.GND, U$8.GND, U$9.GND
- net N$1: now also JP1.2, U$50.P$1; no longer U$3.P$2
- net N$11: now also U$33.2, U$34.2; no longer U$8.CKI
- net N$13: now also U$16.VOUT, U$20.VS, U$28.1; no longer U$18.1, U$8.BFB
- net N$14: now also U$15.VOUT, U$19.VS, U$27.1; no longer U$19.1, U$8.GFB
- net N$15: now also U$18.VS, U$26.1, U$8.VOUT; no longer U$20.1, U$8.RFB
- net N$16: now also T1.E; no longer U$8.SDI
- net N$2: now also U$45.LED1, U$53.EN; no longer U$10.PTA2/JTAG_TDO/TRACE?SWO/EZP_DO/UART0_TX/FTM0_CH7, U$3.P$6
- net N$25: now also U$21.1, U2.VCC
- net N$3: now also U$53.FB, U$54.1, X1-2.S; no longer U$10.PTA1/JTAG_TDI/EZP_DI/UART0/RX/FTM0_CH6, U$3.P$8
- net N$35: now also U$14.D-, U$3.USB0_DM, U$9.2; no longer U$10.PTE17/ADC0_SE5A/SPI0_SCK/UART2_RX/FTM_CLKIN1/LPTMR0_ALT3, U$15.4, U$27.1
- net N$36: now also U$13.2, U$14.D+, U$3.USB0_DP; no longer U$10.PTE4/LLWU_P2/SPI1_PCS0/MTRACE_D0, U$14.4, U$28.1
- net N$37: now also U$20.REXT, U$28.2; no longer U$10.PTE16/ADC0_SE4A/SPI0_PCS0/UART2_TX/FTM_CLKIN0/FTM0_FLT3, U$13.4, U$29.1
- net N$39: now also U$36.1
- net N$4: now also JP1.4, U$51.P$1; no longer U$3.P$4
- net N$40: now also U$37.1
- net N$42: now also U$19.REXT, U$27.2; no longer U$10.PTA18/EXTAL0/FTM0_FTL2_FTM_CLKIN0, U$16.4, U$26.1
- net N$43: now also U$18.REXT, U$26.2; no longer U$36.EN, U$37.EN, U$44.EN, U$45.LED0, U$46.2
- net N$44: now also U$16.EN, U$45.LED0, U$8.EN; no longer U$37.SW, U$47.2, U$50.2
- net N$45: now also U$10.PTD2/LLWU_P13/SPI0_SOUT/UART2_RX/I2C0_SCL/GPIO4_BSM_DATA; no longer U$10.PTD2/LLWU_P13/SPI0_SOUT/UART2_RX/I2C0_SDA/GPIO4_BSM_DATA, U$62.SDA
- net N$46: now also U$10.PTA18/EXTAL0/FTM0_FTL2_FTM_CLKIN0; no longer LQH3NPN100NM0L.2, U$36.SW, U$52.2
- net N$47: now also U$10.PTD3/SPI0_SIN/UART2_TX/I2C0_SDA/GPIO5_BSM_CLK; no longer U$10.PTD3/SPI0_SIN/UART2_TX/I2C0_SCL/GPIO5_BSM_CLK, U$62.SCL
- net N$48: now also T1.C, U$33.1, U$44.DIN; no longer U$44.SW, U$49.2, U$51.2
- net N$49: now also T1.B, U$29.2, U$34.1; no longer R10.1, R12.2, U$33.2, U$34.2, U$9.PWR
- net N$5: now also L1.1, U$14.SHIELD; no longer U$1.GREEN, U$8.GOUT
- net N$50: now also D1.A, U$53.SW, U$55.1; no longer U$44.FB, U$58.2
- net N$51: now also U$1.P$3, U$20.OUT, U$20.OUT1, U$20.OUT2; no longer U$44.OUT, U$55.1, U$58.1, U$59.A1
- net N$52: now also JP2.2, U$3.PTA3, U$47.2; no longer U$37.FB, U$57.2
- net N$53: now also U$1.P$2, U$19.OUT, U$19.OUT1, U$19.OUT2; no longer U$37.OUT, U$54.1, U$57.1, U$59.A2
- net N$54: now also D1.C, U$53.OVP, U$56.2, X1-1.S; no longer U$36.OUT, U$53.1, U$56.1, U$59.A3
- net N$55: now also JP2.4, U$3.PTA0; no longer U$36.FB, U$56.2
- net N$56: now also JP2.6, U$3.PTA2; no longer C11.1, R12.1, U$62.VIN+
- net N$57: now also JP2.8, U$3.PTA1; no longer C11.2, R13.1, U$62.VIN-
- net N$6: now also JP1.10, U$3.PTB1, U$52.2; no longer U$3.P$10
- net N$8: now also U$15.EN; no longer U$1.BLUE, U$8.BOUT
- net N$9: now also U$1.P$1, U$18.OUT, U$18.OUT1, U$18.OUT2; no longer U$1.RED, U$8.ROUT
- net V+: now also POSCON.1, POSCON.8, U$5.VOUT; no longer IC1.IN, R10.2, R13.2, U$1.ANODE, U$31.2, U$8.VCC
Other:
- moved on the sheet: U$26, U$27, U$28

Commit message: Updated KW2 footprint in design
Swapped footprint for one with 3mm foam outline
Parts:
- U$10: value KW2_CPU_COMBO -> KW2_CPU_OFFSET; device KW2:KW2_CPU_COMBO -> KW2:KW2_CPU_OFFSET
Changed lines of the file:
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@@
 <grid distance="0.1" unitdist="inch" unit="inch" style="lines" multiple="1" display="no" altdistance="0.01" altunitdist="inch" altunit="inch"/>
 <layers>
-<layer number="1" name="Top" color="4" fill="1" visible="no" active="no"/>
-<layer number="2" name="GRB2" color="1" fill="3" visible="no" active="no"/>
-<layer number="3" name="Route3" color="4" fill="3" visible="no" active="no"/>
-<layer number="4" name="Route4" color="1" fill="4" visible="no" active="no"/>
-<layer number="5" name="Route5" color="4" fill="4" visible="no" active="no"/>
-<layer number="6" name="Route6" color="1" fill="8" visible="no" active="no"/>
-<layer number="7" name="Route7" color="4" fill="8" visible="no" active="no"/>
-<layer number="8" name="Route8" color="1" fill="2" visible="no" active="no"/>
-<layer number="9" name="Route9" color="4" fill="2" visible="no" active="no"/>
-<layer number="10" name="Route10" color="1" fill="7" visible="no" active="no"/>
-<layer number="11" name="Route11" color="4" fill="7" visible="no" active="no"/>
-<layer number="12" name="Route12" color="1" fill="5" visible="no" active="no"/>
-<layer number="13" name="Route13" color="4" fill="5" visible="no" active="no"/>
-<layer number="14" name="Route14" color="1" fill="6" visible="no" active="no"/>
-<layer number="15" name="Route15" color="4" fill="6" visible="no" active="no"/>
-<layer number="16" name="Bottom" color="1" fill="1" visible="no" active="no"/>
-<layer number="17" name="Pads" color="2" fill="1" visible="no" active="no"/>
-<layer number="18" name="Vias" color="2" fill="1" visible="no" active="no"/>
-<layer number="19" name="Unrouted" color="6" fill="1" visible="no" active="no"/>
-<layer number="20" name="Dimension" color="15" fill="1" visible="no" active="no"/>
-<layer number="21" name="tPlace" color="7" fill="1" visible="no" active="no"/>
-<layer number="22" name="bPlace" color="7" fill="1" visible="no" active="no"/>
-<layer number="23" name="tOrigins" color="15" fill="1" visible="no" active="no"/>
-<layer number="24" name="bOrigins" color="15" fill="1" visible="no" active="no"/>
-<layer number="25" name="tNames" color="7" fill="1" visible="no" active="no"/>
-<layer number="26" name="bNames" color="7" fill="1" visible="no" active="no"/>
-<layer number="27" name="tValues" color="7" fill="1" visible="no" active="no"/>
-<layer number="28" name="bValues" color="7" fill="1" visible="no" active="no"/>
+<layer number="1" name="Top" color="4" fill="1" visible="yes" active="no"/>
+<layer number="2" name="GRB2" color="1" fill="3" visible="yes" active="no"/>
+<layer number="3" name="Route3" color="4" fill="3" visible="yes" active="no"/>
+<layer number="4" name="Route4" color="1" fill="4" visible="yes" active="no"/>
+<layer number="5" name="Route5" color="4" fill="4" visible="yes" active="no"/>
+<layer number="6" name="Route6" color="1" fill="8" visible="yes" active="no"/>
+<layer number="7" name="Route7" color="4" fill="8" visible="yes" active="no"/>
+<layer number="8" name="Route8" color="1" fill="2" visible="yes" active="no"/>
+<layer number="9" name="Route9" color="4" fill="2" visible="yes" active="no"/>
+<layer number="10" name="Route10" color="1" fill="7" visible="yes" active="no"/>
+<layer number="11" name="Route11" color="4" fill="7" visible="yes" active="no"/>
+<layer number="12" name="Route12" color="1" fill="5" visible="yes" active="no"/>
+<layer number="13" name="Route13" color="4" fill="5" visible="yes" active="no"/>
+<layer number="14" name="Route14" color="1" fill="6" visible="yes" active="no"/>
+<layer number="15" name="Route15" color="4" fill="6" visible="yes" active="no"/>
+<layer number="16" name="Bottom" color="1" fill="1" visible="yes" active="no"/>
+<layer number="17" name="Pads" color="2" fill="1" visible="yes" active="no"/>
+<layer number="18" name="Vias" color="2" fill="1" visible="yes" active="no"/>
+<layer number="19" name="Unrouted" color="6" fill="1" visible="yes" active="no"/>
+<layer number="20" name="Dimension" color="15" fill="1" visible="yes" active="no"/>
+<layer number="21" name="tPlace" color="7" fill="1" visible="yes" active="no"/>
+<layer number="22" name="bPlace" color="7" fill="1" visible="yes" active="no"/>
+<layer number="23" name="tOrigins" color="15" fill="1" visible="yes" active="no"/>
+<layer number="24" name="bOrigins" color="15" fill="1" visible="yes" active="no"/>
+<layer number="25" name="tNames" color="7" fill="1" visible="yes" active="no"/>
+<layer number="26" name="bNames" color="7" fill="1" visible="yes" active="no"/>
+<layer number="27" name="tValues" color="7" fill="1" visible="yes" active="no"/>
+<layer number="28" name="bValues" color="7" fill="1" visible="yes" active="no"/>
 <layer number="29" name="tStop" color="7" fill="3" visible="no" active="no"/>
 <layer number="30" name="bStop" color="7" fill="6" visible="no" active="no"/>
@@
 <layer number="35" name="tGlue" color="7" fill="4" visible="no" active="no"/>
 <layer number="36" name="bGlue" color="7" fill="5" visible="no" active="no"/>
-<layer number="37" name="tTest" color="7" fill="1" visible="no" active="no"/>
-<layer number="38" name="bTest" color="7" fill="1" visible="no" active="no"/>
+<layer number="37" name="tTest" color="7" fill="1" visible="yes" active="no"/>
+<layer number="38" name="bTest" color="7" fill="1" visible="yes" active="no"/>
 <layer number="39" name="tKeepout" color="4" fill="11" visible="no" active="no"/>
 <layer number="40" name="bKeepout" color="1" fill="11" visible="no" active="no"/>
@@
 <layer number="44" name="Drills" color="7" fill="1" visible="no" active="no"/>
 <layer number="45" name="Holes" color="7" fill="1" visible="no" active="no"/>
-<layer number="46" name="Milling" color="3" fill="1" visible="no" active="no"/>
-<layer number="47" name="Measures" color="7" fill="1" visible="no" active="no"/>
-<layer number="48" name="Document" color="7" fill="1" visible="no" active="no"/>
-<layer number="49" name="Reference" color="7" fill="1" visible="no" active="no"/>
-<layer number="50" name="dxf" color="7" fill="1" visible="no" active="no"/>
-<layer number="51" name="tDocu" color="7" fill="1" visible="no" active="no"/>
-<layer number="52" name="bDocu" color="7" fill="1" visible="no" active="no"/>
-<layer number="53" name="tGND_GNDA" color="7" fill="1" visible="no" active="no"/>
-<layer number="54" name="bGND_GNDA" color="7" fill="1" visible="no" active="no"/>
-<layer number="56" name="wert" color="7" fill="1" visible="no" active="no"/>
-<layer number="57" name="tCAD" color="7" fill="1" visible="no" active="no"/>
+<layer number="46" name="Milling" color="3" fill="1" visible="yes" active="no"/>
+<layer number="47" name="Measures" color="7" fill="1" visible="yes" active="no"/>
+<layer number="48" name="Document" color="7" fill="1" visible="yes" active="no"/>
+<layer number="49" name="Reference" color="7" fill="1" visible="yes" active="no"/>
+<layer number="50" name="dxf" color="7" fill="1" visible="yes" active="no"/>
+<layer number="51" name="tDocu" color="7" fill="1" visible="yes" active="no"/>
+<layer number="52" name="bDocu" color="7" fill="1" visible="yes" active="no"/>
+<layer number="53" name="tGND_GNDA" color="7" fill="1" visible="yes" active="no"/>
+<layer number="54" name="bGND_GNDA" color="7" fill="1" visible="yes" active="no"/>
+<layer number="56" name="wert" color="7" fill="1" visible="yes" active="no"/>
+<layer number="57" name="tCAD" color="7" fill="1" visible="yes" active="no"/>
 <layer number="91" name="Nets" color="2" fill="1" visible="yes" active="yes"/>
 <layer number="92" name="Busses" color="1" fill="1" visible="yes" active="yes"/>
@@
 </classes>
 <parts>
-<part name="U$10" library="KW2" deviceset="KW2_CPU" device="_COMBO" value="KW2_CPU_COMBO"/>
+<part name="U$10" library="KW2" deviceset="KW2_CPU" device="_OFFSET" value="KW2_CPU_OFFSET"/>
 <part name="POSCON" library="GW-devices" deviceset="RJ45-8" device="" value="">
 <attribute name="MFGN" value="Molex"/>
